Commit message: moving object in moving bin

File: content/assets/urdf/mug/movable_mug.urdf (robot description, URDF)
Before this commit: robot mug, 7 links, 6 joints
Links:
- link mug: mass 0.0 -> None

File: content/assets/urdf/mug/mug.urdf (robot description, URDF)
Before this commit: robot mug, 1 links, 0 joints
Links:
- link mug: mass 0.102 -> None; geometry visual mesh filename=mug.obj scale=1 1 1
